File: mainboard/mainboard.kicad_sch (KiCad schematic)
At the start: 0 parts

Commit message: Added basic components
Parts:
- added A1: Raspberry Pi Zero, symbol GTMRG-Boards:RPi_Zero_2
- added A2: Adafruit ICM-20948 9DoF IMU, symbol GTMRG-Boards:Adafruit_ICM-20948
- added A3: MakerFocus GT-U7 GPS, symbol GTMRG-Boards:MakerFocus_GT-U7
Connections:
- new net GND: A1.14 (GND), A1.20 (GND), A1.25 (GND), A1.30 (GND), A1.34 (GND), A1.39 (GND), A1.6 (GND), A1.9 (GND), A2.11 (GND), A2.2 (GND), A3.1 (GND)

Commit message: Updated mainboard
Parts:
- added J1: Port ESC Connector, symbol Connector:Conn_01x03_Pin
- added J2: Stbd ESC Connector, symbol Connector:Conn_01x03_Pin
- added JP1: P_Jumper, symbol Jumper:SolderJumper_3_Open
- added JP2: S_Jumper, symbol Jumper:SolderJumper_3_Open
Connections:
- net GND: now also J1.3 (Pin_3), J2.3 (Pin_3)
- net GPS_TX: now reaches A1.10 (GP15_UART0_RX)
- net GPS_TX: now also A3.3 (TXD)
- net +5V_P: now reaches A1.2 (5V)
- net +5V_P: now also JP1.2 (C)
- net SDA: now reaches A1.3 (GP2_SDA_I2C)
- net SDA: now also A2.4 (SDA)
- net SCL: now reaches A1.5 (GP3_SCL_I2C)
- net SCL: now also A2.3 (SCL)
- net GPS_RX: now reaches A1.8 (GP14_UART0_TX)
- net GPS_RX: now also A3.2 (RXD)
- net +5V_S: now reaches A3.0 (VCC)
- net +5V_S: now also A2.0 (VIN), JP2.2 (C)
- new net +5V_PEsc: J1.2 (Pin_2), JP1.1 (A)
- new net +5V_Reg: JP1.3 (B), JP2.1 (A)
- new net +5V_SEsc: J2.2 (Pin_2), JP2.3 (B)
- new net PEsc_Sig: J1.1 (Pin_1)
- new net SEsc_Sig: J2.1 (Pin_1)
- no-connect marks 0 -> 8
Other:
- moved on the sheet: A1, A2, A3
